File: ARES_FC.kicad_pcb (KiCad board)
At the start: 2 copper layers, 57.2 x 57.2 mm, 67 parts, among them J1 SWD, J2 TYPE-C-31-M-12, J3 FC_M/P, J4 5V, J5 GND, J6 FC_RF, J7 Conn_01x04_Pin, J8 Conn_01x04_Pin, U1 STM32F401CCU6, U2 AMS1117-3.3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

Commit message: TVS diodes WIP
Parts:
- removed C1: 100nF, Capacitor_SMD:C_0402_1005Metric
- added D5: RCLAMP0502B, Package_TO_SOT_SMD:SOT-416, F.Cu at (169.4, 94.3)
- added D6: RCLAMP0502B, Package_TO_SOT_SMD:SOT-416, F.Cu at (132.9, 77.2)
- added D7: RCLAMP0502B, Package_TO_SOT_SMD:SOT-416, F.Cu at (159.9, 73.1)
- added U7: CDSOT236-0504C, Package_TO_SOT_SMD:SOT-23-6, F.Cu at (127.8, 96.9)
- moved J7 2.14 mm to (161.9, 77.7)
Routing:
- net /SCL: track 65.9 -> 76.8 mm, vias 6 -> 7
- net /SDA: track 62.9 -> 72.6 mm
- net /USB_D-: track 24.8 -> 28.3 mm
- net /NRST: track 32.7 -> 30.0 mm
- net +3.3V: track 234.9 -> 232.2 mm
- net /USB_D+: track 25.2 -> 27.6 mm
- net GND: track 81.0 -> 79.6 mm, vias 403 -> 394
