File: ARES_FC.kicad_sch (KiCad schematic)
At the start: 65 parts, among them J1 SWD, J2 TYPE-C-31-M-12, J3 FC_M/P, J4 5V, J5 GND, J6 FC_RF, J7 Conn_01x04_Pin, J8 Conn_01x04_Pin, U1 STM32F401CCU6, U2 AMS1117-3.3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

Commit message: TVS diodes WIP
Parts:
- added D5, D6, D7, D8, D9: RCLAMP0502B, Package_TO_SOT_SMD:SOT-416, symbol Power_Protection:RCLAMP0502B
Connections:
- net GND: now also D5.3 (A), D6.3 (A), D7.3 (A), D8.3 (A), D9.3 (A)
- net NRST: now also D9.2 (K2)
- net SCL: now also D6.1 (K1), D7.2 (K2)
- net SDA: now also D6.2 (K2), D7.1 (K1)
- net SWCLK: now also D8.2 (K2)
- net SWDIO: now also D8.1 (K1)
- net USB_D+: now also D5.2 (K2)
- net USB_D-: now also D5.1 (K1)
- no-connect marks 19 -> 20
Other:
- moved on the sheet: J1, J2, R1, R2
